File: main/untitled.brd (EAGLE design)
At the start: 68 x 64.9 mm, 30 parts, among them IC1 MCP1700, Q1 8MHz

Commit message: ultimate version
Parts:
- removed C5, C6: 1µ, rcl:C0603
- removed C7: 4.7µ, rcl:C0603
- removed C8: 10n, rcl:C0603
- removed IC1: MCP1700, linear:SOT23
- removed Q1: 8MHz, special:QS
- removed R2: 100-400R ?, rcl:R0603
- removed SJ2: 0R, rcl:R0201
- removed SV3: (no value), con-lstb:MA13-1
- removed SV4: (no value), con-lstb:MA05-1
- added C5**1: (no value), rcl:C0603
- added C9: 100n/35V, rcl:C0805
- added DRILEGEND: (no value), drilegend:DRILEGEND
- added NUCLEO_ISP: (no value), con-lstb:MA05-1
- added U$3: (no value), _biblioteka_1:LOGO_SMALL
- added U$4: HT7333, _biblioteka_1:SOT89
- C2: value 100n -> 10µ
- C3: value 16p -> 22µ/16V; device rcl:C0603 -> adafruit:E2,5-6
- C4: value 16p -> 10µ/10V
- C5**: value (none) -> 100-200n
- moved R1 59.4 mm to (35.7, 40.9), turned to 180 degrees
- moved SV5 41.5 mm to (30.1, 18.5), turned to 180 degrees
- moved S1 30.9 mm to (53.7, 53.7), flipped to the bottom
- moved U$2 22.8 mm to (21.3, 53.5)
- moved R1* 13.6 mm to (25.4, 35.4), turned to 180 degrees
- moved SJ1 9.69 mm to (42.4, 52.2)
- moved C4 9.05 mm to (34.9, 48.1), turned to 180 degrees
- moved C2 7.94 mm to (39.7, 36.4), flipped to the bottom, turned to 0 degrees
- moved C3 7.75 mm to (21.8, 43.3), turned to 180 degrees
- moved C5** 4.03 mm to (30.9, 33.6), turned to 270 degrees
- moved C1 3.77 mm to (35.2, 36.1), flipped to the bottom, turned to 180 degrees
- moved SV6 2.85 mm to (56.5, 26.1), turned to 270 degrees
- moved U$1 2.47 mm to (37.7, 35.8)
Connections:
- removed net AGND: SJ2.1, SV2.3
- removed net N$10: U$1.18
- removed net N$13: U$1.14
- removed net N$2: U$1.7
- removed net N$3: C3.2, Q1.1, R2.1
- removed net N$5: R2.2, U$1.3
- removed net V+LDR: SV2.2
- removed net V+LED: SV2.5
- removed net V+LOGIC: SV1.1
- removed net VW_VCC: SJ1.2, SV6.2
- new net BTN: S1.2, U$1.18
- net +3V3: now also C4.1, NUCLEO_ISP.1, SV1.1, SV2.2, U$4.3; no longer C6.1, C7.1, C8.1, IC1.2, SV4.1
- net GND: now also C3.-, C4.2, C5**1.2, C9.2, NUCLEO_ISP.3, SV2.3, U$4.1; no longer C3.1, C4.1, C5.2, C6.2, C7.2, C8.2, IC1.1, SJ2.2, SV4.5
- net N$1: now also SJ1.2, SV6.3; no longer C4.2, Q1.2, U$1.2
- net N$4: now also C5**1.1
- net NRST: now also NUCLEO_ISP.5; no longer SV4.2
- net SWCLK: now also NUCLEO_ISP.2; no longer SV4.4
- net SWDIO: now also NUCLEO_ISP.4; no longer SV4.3
- net V+: now also C3.+, C9.1, SV2.5, U$4.2, U$4.2.1; no longer C5.1, IC1.3
- net VW_IN: now also SV6.2, U$1.14; no longer SV6.3
Routing:
- net +3V3: track 0.00 -> 159.4 mm, vias 0 -> 3
- net V+: track 0.00 -> 59.5 mm, vias 0 -> 2
- net N$1: track 0.00 -> 59.3 mm, vias 0 -> 1
- net BTN: track 0.00 -> 40.6 mm, vias 0 -> 1
- net TX: track 0.00 -> 23.7 mm
- net NRST: track 0.00 -> 21.8 mm, vias 0 -> 1
- net RX: track 0.00 -> 21.3 mm
- net LDR: track 0.00 -> 20.3 mm
- net VW_IN: track 0.00 -> 19.5 mm
- net SDI: track 0.00 -> 16.4 mm
- net SWCLK: track 0.00 -> 16.1 mm
- net OE: track 0.00 -> 15.1 mm
- net LA: track 0.00 -> 14.0 mm
- net CLK: track 0.00 -> 13.7 mm
- net N$4: track 0.00 -> 10.7 mm
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- added copper zone on layer 1, net +3V3
- added copper zone on layer 1, net GND
- added copper zone on layer 16, net GND
- added copper zone on layer 1, net V+
Other:
- outline, holes or cut-outs redrawn
- board text added: "+"
- board text added: "+3v3"
- board text added: "+V"
- board text added: "01-16"
- board text added: "01-20"
- board text added: ">PLOT_DATE_TIME"
- board text added: "GND"
- board text added: "Krawędź polygonu masy odsunięta od krawędzi PCB"
- board text added: "LAYER-STACK"
- board text added: "Otwór środkowy - 7.5mm"
- board text added: "Rx"
- board text added: "Tx"
- board text added: "krawędź PCB"
- board text added: "linia lutowania złącza"
- board text added: "otwory na śruby mocujące - 3mm lub 2.5mm przy zachowaniu precyzji"
- board text removed: "krawędź PCB (jeszcze sprawdź)"
- board text removed: "linia lutowania złącza (jeszcze sprawdź)"
