File: main/untitled.sch (EAGLE design)
At the start: 30 parts, among them IC1 MCP1700, Q1 8MHz

Commit message: ultimate version
Parts:
- removed C5, C6: 1µ, rcl:C-EUC0603
- removed C7: 4.7µ, rcl:C-EUC0603
- removed C8: 10n, rcl:C-EUC0603
- removed IC1: MCP1700, linear:MCP1703CB
- removed Q1: 8MHz, special:XTAL/S
- removed R2: 100-400R ?, rcl:R-EU_R0603
- removed SJ2: 0R, rcl:R-EU_R0201
- removed SV3: (no value), con-lstb:MA13-1
- removed SV4: (no value), con-lstb:MA05-1
- added C5**1: (no value), rcl:C-EUC0603
- added C9: 100n/35V, rcl:C-EUC0805
- added NUCLEO_ISP: (no value), con-lstb:MA05-1
- added U$4: HT7333, _biblioteka_1:HT7333
- C2: value 100n -> 10µ
- C3: value 16p -> 22µ/16V; device rcl:C-EUC0603 -> adafruit:CPOL-USE2.5-6
- C4: value 16p -> 10µ/10V
- C5**: value (none) -> 100-200n
Connections:
- removed net AGND: SJ2.1, SV2.3
- removed net N$10: U$1.PA10
- removed net N$13: U$1.PB1
- removed net N$2: U$1.PA1
- removed net N$3: C3.2, Q1.1, R2.1
- removed net N$5: R2.2, U$1.PF1-OSC_OUT
- removed net V+LDR: SV2.2
- removed net V+LED: SV2.5
- removed net V+LOGIC: SV1.1
- removed net VW_VCC: SJ1.2, SV6.2
- new net BTN: S1.S, U$1.PA10
- net +3V3: now also C4.1, NUCLEO_ISP.1, SV1.1, SV2.2, U$4.VOUT; no longer C6.1, C7.1, C8.1, IC1.VO, SV4.1
- net GND: now also C3.-, C4.2, C5**1.2, C9.2, NUCLEO_ISP.3, SV2.3, U$4.GND; no longer C3.1, C4.1, C5.2, C6.2, C7.2, C8.2, IC1.GND, SJ2.2, SV4.5
- net N$1: now also SJ1.2, SV6.3; no longer C4.2, Q1.2, U$1.PF0-OSC_IN
- net N$4: now also C5**1.1
- net NRST: now also NUCLEO_ISP.5; no longer SV4.2
- net SWCLK: now also NUCLEO_ISP.2; no longer SV4.4
- net SWDIO: now also NUCLEO_ISP.4; no longer SV4.3
- net V+: now also C3.+, C9.1, SV2.5, U$4.VIN; no longer C5.1, IC1.VI
- net VW_IN: now also SV6.2, U$1.PB1; no longer SV6.3
Other:
- note added: "V+LDR"
- note added: "V+LED"
- note added: "V+LOGIC"
- moved on the sheet: C4, SJ1
